Commit message: Path planning is fixed but PID gains still need tuning

File: src/onrobot/onrobot_rg_description/urdf/onrobot_rg2_gazebo.xacro (robot description, xacro)
@@ -2,10 +2,10 @@
 <robot xmlns:xacro="http://ros.org/wiki/xacro">
   <xacro:macro name="onrobot_rg2_gazebo" params="prefix">
-    <gazebo>
+    <!--gazebo>
       <plugin name="gazebo_ros_control" filename="libgazebo_ros_control.so">
         <robotNamespace>/onrobot_rg2</robotNamespace>
         <robotSimType>gazebo_ros_control/DefaultRobotHWSim</robotSimType>
       </plugin>
-    </gazebo>
+    </gazebo-->
     <gazebo>
       <plugin filename="libroboticsgroup_upatras_gazebo_mimic_joint_plugin.so" name="mimic_${prefix}left_inner_knuckle_joint">

File: src/onrobot/onrobot_rg_description/urdf/onrobot_rg2_transmission.xacro (robot description, xacro)
@@ -5,8 +5,8 @@
       <type>transmission_interface/SimpleTransmission</type>
       <joint name="${prefix}finger_joint">
-        <hardwareInterface>hardware_interface/EffortJointInterface</hardwareInterface>
+        <hardwareInterface>hardware_interface/PositionJointInterface</hardwareInterface>
       </joint>
       <actuator name="${prefix}finger_joint_motor">
-        <hardwareInterface>hardware_interface/EffortJointInterface</hardwareInterface>
+        <hardwareInterface>hardware_interface/PositionJointInterface</hardwareInterface>
         <mechanicalReduction>1</mechanicalReduction>
       </actuator>

File: src/ur10e_sim/urdf/ur10e_workarea.urdf.xacro (robot description, xacro)
@@ -20,6 +20,6 @@
     <inertial>
       <origin xyz="0 0 0" rpy="0 0 0"/>
-      <mass value="10.0"/>
-      <inertia ixx="0.84" ixy="0" ixz="0" iyy="0.84" iyz="0" izz="1.67" />
+      <mass value="100.0"/>
+      <inertia ixx="8.4" ixy="0" ixz="0" iyy="8.4" iyz="0" izz="16.7" />
     </inertial>
   </link>
@@ -40,8 +40,17 @@
     <child link="base_link"/> <origin xyz="0 0 0.05" rpy="0 0 0"/>
   </joint>
+  <gazebo reference="table_to_robot">
+    <preserveFixedJoint>true</preserveFixedJoint>
+  </gazebo>
   <xacro:onrobot_rg2 prefix=""/>
   <joint name="gripper_attachment" type="fixed">
   <parent link="tool0"/> <child link="onrobot_rg2_base_link"/>
   <origin xyz="0 0 0" rpy="0 0 1.5708"/>
+  </joint>
+  <link name="gripper_tcp"/>
+  <joint name="gripper_tcp_attachment" type="fixed">
+    <parent link="onrobot_rg2_base_link"/>
+    <child link="gripper_tcp"/>
+    <origin xyz="0 0 0.15" rpy="0 0 0"/>
   </joint>
   <gazebo>
@@ -51,3 +60,25 @@
     </plugin>
   </gazebo>
+  <gazebo reference="wrist_3_joint">
+  <implicitSpringDamper>true</implicitSpringDamper>
+  <kp>1000000.0</kp>
+  <kd>100.0</kd>
+</gazebo>
+<gazebo reference="shoulder_pan_joint">   <implicitSpringDamper>true</implicitSpringDamper> </gazebo>
+<gazebo reference="shoulder_lift_joint">  <implicitSpringDamper>true</implicitSpringDamper> </gazebo>
+<gazebo reference="elbow_joint">          <implicitSpringDamper>true</implicitSpringDamper> </gazebo>
+<gazebo reference="wrist_1_joint">        <implicitSpringDamper>true</implicitSpringDamper> </gazebo>
+<gazebo reference="wrist_2_joint">        <implicitSpringDamper>true</implicitSpringDamper> </gazebo>
+<gazebo>
+  <physics type="ode">
+    <max_step_size>0.001</max_step_size>
+    <real_time_update_rate>1000</real_time_update_rate>
+    <ode>
+      <solver>
+        <type>quick</type>
+        <iters>100</iters>
+      </solver>
+    </ode>
+  </physics>
+</gazebo>
 </robot>
