Commit message: pick and place task working..path planning should be optimized

File: src/onrobot/onrobot_rg_description/urdf/onrobot_rg2_model_macro.xacro (robot description, xacro)
@@ -103,5 +103,5 @@
       <child link="${prefix}${fingerprefix}_inner_knuckle" />
       <axis xyz="1 0 0" />
-      <limit lower="-0.785398" upper="0.785398" velocity="100.0" effort="1000" />
+      <limit lower="-1" upper="1" velocity="100.0" effort="1000" />
       <mimic joint="${prefix}finger_joint" multiplier="-1" offset="0" />
     </joint>
@@ -113,5 +113,5 @@
       <child link="${prefix}${fingerprefix}_inner_finger" />
       <axis xyz="1 0 0" />
-      <limit lower="-0.872665" upper="0.872665" velocity="100.0" effort="1000" />
+      <limit lower="-1" upper="1" velocity="100.0" effort="1000" />
       <mimic joint="${prefix}finger_joint" multiplier="1" offset="0" />
     </joint>
@@ -124,5 +124,5 @@
       <child link="${prefix}left_outer_knuckle" />
       <axis xyz="-1 0 0" />
-      <limit lower="-0.558505" upper="0.785398" velocity="100.0" effort="1000" />
+      <limit lower="-1" upper="1" velocity="100.0" effort="1000" />
     </joint>
     <xacro:finger_joints prefix="${prefix}" fingerprefix="left" reflect="1.0"/>
@@ -134,5 +134,5 @@
       <child link="${prefix}right_outer_knuckle" />
       <axis xyz="1 0 0" />
-      <limit lower="-0.785398" upper="0.785398" velocity="100.0" effort="1000" />
+      <limit lower="-1" upper="1" velocity="100.0" effort="1000" />
       <mimic joint="${prefix}finger_joint" multiplier="-1" offset="0" />
     </joint>

File: src/ur10e_sim/urdf/ur10e_workarea.urdf.xacro (robot description, xacro)
@@ -82,10 +82,14 @@
     <origin xyz="0 0 0" rpy="0 0 0"/>
   </joint>
-  <gazebo>
-    <plugin name="gazebo_ros_control" filename="libgazebo_ros_control.so">
-      <robotNamespace>/</robotNamespace>
-      <robotSimType>gazebo_ros_control/DefaultRobotHWSim</robotSimType>
-    </plugin>
-  </gazebo>
+<gazebo>
+  <plugin name="gazebo_ros_link_attacher" filename="libgazebo_ros_link_attacher.so"/>
+  <plugin name="gazebo_ros_api_plugin" filename="libgazebo_ros_api_plugin.so"/>
+</gazebo>
+<gazebo>
+  <plugin name="gazebo_ros_control" filename="libgazebo_ros_control.so">
+    <robotNamespace>/</robotNamespace>
+    <robotSimType>gazebo_ros_control/DefaultRobotHWSim</robotSimType>
+  </plugin>
+</gazebo>
   <gazebo reference="wrist_3_joint">
   <implicitSpringDamper>true</implicitSpringDamper>
