Commit message: moveit launch file added

File: src/ur10e_sim/urdf/ur10e_workarea.urdf.xacro (robot description, xacro)
@@ -18,4 +18,9 @@
       </geometry>
     </collision>
+    <inertial>
+      <origin xyz="0 0 0" rpy="0 0 0"/>
+      <mass value="10.0"/>
+      <inertia ixx="0.84" ixy="0" ixz="0" iyy="0.84" iyz="0" izz="1.67" />
+    </inertial>
   </link>
   <joint name="world_to_table" type="fixed">
@@ -40,3 +45,9 @@
   <origin xyz="0 0 0" rpy="0 0 1.5708"/>
   </joint>
+  <gazebo>
+    <plugin name="gazebo_ros_control" filename="libgazebo_ros_control.so">
+      <robotNamespace>/</robotNamespace>
+      <robotSimType>gazebo_ros_control/DefaultRobotHWSim</robotSimType>
+    </plugin>
+  </gazebo>
 </robot>

Commit message: tables and object for pick and place added

File: src/ur10e_sim/urdf/ur10e_workarea.urdf.xacro (robot description, xacro)
@@ -3,6 +3,7 @@
   <xacro:include filename="$(find ur_description)/urdf/inc/ur_macro.xacro"/>
   <xacro:include filename="$(find onrobot_rg_description)/urdf/onrobot_rg2_model_macro.xacro" />
+  <xacro:include filename="$(find ur10e_sim)/urdf/table.urdf.xacro" />
   <link name="world"/>
-  <link name="table">
+  <link name="floor_plate">
     <visual>
       <geometry>
@@ -24,7 +25,7 @@
     </inertial>
   </link>
-  <joint name="world_to_table" type="fixed">
+  <joint name="world_to_floor_plate" type="fixed">
     <parent link="world"/>
-    <child link="table"/>
+    <child link="floor_plate"/>
     <origin xyz="0 0 0.05" rpy="0 0 0"/>
   </joint>
@@ -37,5 +38,5 @@
   />
   <joint name="table_to_robot" type="fixed">
-    <parent link="table"/>
+    <parent link="floor_plate"/>
     <child link="base_link"/> <origin xyz="0 0 0.05" rpy="0 0 0"/>
   </joint>
@@ -53,4 +54,16 @@
     <child link="gripper_tcp"/>
     <origin xyz="0 0 0.15" rpy="0 0 0"/>
+  </joint>
+  <xacro:wooden_table prefix="right_"/>
+  <joint name="right_table_attachment" type="fixed">
+    <parent link="world"/>
+    <child link="right_table_base_link"/>
+    <origin xyz="0 1 0" rpy="0 0 0"/>
+  </joint>
+  <xacro:wooden_table prefix="left_"/>
+  <joint name="left_table_attachment" type="fixed">
+    <parent link="world"/>
+    <child link="left_table_base_link"/>
+    <origin xyz="0 -1 0" rpy="0 0 0"/>
   </joint>
   <gazebo>

Commit message: FT sensor added, collisions still need to be updated

File: src/ur10e_sim/urdf/ur10e_workarea.urdf.xacro (robot description, xacro)
@@ -4,4 +4,6 @@
   <xacro:include filename="$(find onrobot_rg_description)/urdf/onrobot_rg2_model_macro.xacro" />
   <xacro:include filename="$(find ur10e_sim)/urdf/table.urdf.xacro" />
+  <xacro:include filename="$(find ur10e_sim)/urdf/tool_adapter_plate.xacro" />
+  <xacro:include filename= "$(find ur10e_sim)/urdf/FT_sensor_urdf/net_ft_sensor_macro.urdf.xacro" />
   <link name="world"/>
   <link name="floor_plate">
@@ -44,7 +46,13 @@
     <preserveFixedJoint>true</preserveFixedJoint>
   </gazebo>
+  <xacro:adapter_plate parent="tool0" prefix="">
+    <origin xyz="0 0 0" rpy="0 0 0"/>
+  </xacro:adapter_plate>
+  <xacro:net_ft_sensor parent="adapter_plate_socket" prefix="">
+    <origin xyz="0 0 0" rpy="0 0 0"/>
+  </xacro:net_ft_sensor>
   <xacro:onrobot_rg2 prefix=""/>
   <joint name="gripper_attachment" type="fixed">
-  <parent link="tool0"/> <child link="onrobot_rg2_base_link"/>
+  <parent link="tool_mount_link"/> <child link="onrobot_rg2_base_link"/>
   <origin xyz="0 0 0" rpy="0 0 1.5708"/>
   </joint>
