Commit message: Gripper controllers fixed

File: src/ur10e_sim/urdf/table.urdf.xacro (robot description, xacro)
@@ -6,5 +6,5 @@
 <xacro:macro name="wooden_table" params="prefix">
 <xacro:property name="table_height" value="0.7" />
-    <xacro:property name="table_width" value="1.0" />
+    <xacro:property name="table_width" value="2.0" />
     <xacro:property name="table_depth" value="0.8" />
     <xacro:property name="leg_radius" value="0.02" />

Commit message: pallette and lebkuchen added..need to fix the planning getting aborted

File: src/ur10e_sim/urdf/table.urdf.xacro (robot description, xacro)
@@ -49,4 +49,10 @@
     <xacro:table_leg leg_suffix="back_left"   x="${-table_width/2 + 0.05}" y="${table_depth/2 - 0.05}" />
     <xacro:table_leg leg_suffix="back_right"  x="${-table_width/2 + 0.05}" y="${-table_depth/2 + 0.05}" />
+    <link name="${prefix}pallette_mount_link"/>
+    <joint name="${prefix}pallette_attachment" type="fixed">
+      <parent link="${prefix}table_top"/>
+      <child link="${prefix}pallette_mount_link"/>
+      <origin xyz="0 0 ${top_thickness/2}" rpy="0 0 0"/>
+    </joint>
     <gazebo reference="${prefix}table_top">
       <material>Gazebo/Wood</material>

File: src/ur10e_sim/urdf/ur10e_workarea.urdf.xacro (robot description, xacro)
@@ -6,4 +6,5 @@
   <xacro:include filename="$(find ur10e_sim)/urdf/tool_adapter_plate.xacro" />
   <xacro:include filename= "$(find ur10e_sim)/urdf/FT_sensor_urdf/net_ft_sensor_macro.urdf.xacro" />
+  <xacro:include filename="$(find ur10e_sim)/urdf/pallette.urdf.xacro" />
   <link name="world"/>
   <link name="floor_plate">
@@ -75,4 +76,10 @@
     <origin xyz="0 -1 0" rpy="0 0 0"/>
   </joint>
+  <xacro:wooden_pallette prefix=""/>
+  <joint name="pallette_attachment" type="fixed">
+    <parent link="right_pallette_mount_link"/>
+    <child link="pallette"/>
+    <origin xyz="0 0 0" rpy="0 0 0"/>
+  </joint>
   <gazebo>
     <plugin name="gazebo_ros_control" filename="libgazebo_ros_control.so">
