Commit message: robot positioned in front of the kuchen

File: src/ur10e_sim/urdf/lebkuchen.urdf.xacro (robot description, xacro)
@@ -3,10 +3,10 @@
   <link name="package_link">
     <inertial>
-      <origin xyz="0 0 0.05" rpy="0 0 0" />
+      <origin xyz="0 0 0.05" rpy="0 0 1.57" />
       <mass value="0.5" />
       <inertia ixx="0.0012" ixy="0" ixz="0" iyy="0.0015" iyz="0" izz="0.0018" />
     </inertial>
     <visual>
-      <origin xyz="0 0 0" rpy="0 0 0" />
+      <origin xyz="0 0 0" rpy="0 0 1.57" />
       <geometry>
         <mesh filename="package://ur10e_sim/meshes/Lebkuchen.stl" scale="0.001 0.001 0.001" />
@@ -15,5 +15,5 @@
     </visual>
     <collision>
-      <origin xyz="0 0 0" rpy="0 0 0" />
+      <origin xyz="0 0 0" rpy="0 0 1.57" />
       <geometry>
         <mesh filename="package://ur10e_sim/meshes/Lebkuchen.stl" scale="0.001 0.001 0.001" />
@@ -44,5 +44,5 @@
     <parent link="package_link"/>
     <child link="kuchen_link"/>
-    <origin xyz="0.0 0.0 0.02" rpy="0 0 0"/>
+    <origin xyz="0.0 0.0 0.02" rpy="0 0 1.57"/>
   </joint>
 <gazebo reference="package_link">

File: src/ur10e_sim/urdf/table.urdf.xacro (robot description, xacro)
@@ -5,6 +5,6 @@
   </material>
 <xacro:macro name="wooden_table" params="prefix">
-<xacro:property name="table_height" value="0.7" />
-    <xacro:property name="table_width" value="2.0" />
+<xacro:property name="table_height" value="0.8" />
+    <xacro:property name="table_width" value="1.5" />
     <xacro:property name="table_depth" value="0.8" />
     <xacro:property name="leg_radius" value="0.02" />

Commit message: camera added..lebkuchen pedestal added

File: src/ur10e_sim/urdf/lebkuchen.urdf.xacro (robot description, xacro)
@@ -49,8 +49,8 @@
     <visual>
       <material>
-        <ambient>0 0.39 0 1</ambient>
-        <diffuse>0 0.39 0 1</diffuse>
-        <specular>0.1 0.1 0.1 1</specular>
-        <emissive>0 0 0 0</emissive>
+        <ambient>0.0 0.6 0.0 1</ambient>
+        <diffuse>0.0 0.8 0.0 1</diffuse>
+        <specular>0.3 0.3 0.3 1</specular>
+        <emissive>0.0 0.0 0.0 0</emissive>
       </material>
     </visual>

File: src/ur10e_sim/urdf/table.urdf.xacro (robot description, xacro)
@@ -49,8 +49,8 @@
     <xacro:table_leg leg_suffix="back_left"   x="${-table_width/2 + 0.05}" y="${table_depth/2 - 0.05}" />
     <xacro:table_leg leg_suffix="back_right"  x="${-table_width/2 + 0.05}" y="${-table_depth/2 + 0.05}" />
-    <link name="${prefix}pallette_mount_link"/>
-    <joint name="${prefix}pallette_attachment" type="fixed">
+    <link name="${prefix}table_mount_link"/>
+    <joint name="${prefix}table_attachment_joint" type="fixed">
       <parent link="${prefix}table_top"/>
-      <child link="${prefix}pallette_mount_link"/>
+      <child link="${prefix}table_mount_link"/>
       <origin xyz="0 0 ${top_thickness/2}" rpy="0 0 0"/>
     </joint>

File: src/ur10e_sim/urdf/ur10e_workarea.urdf.xacro (robot description, xacro)
@@ -7,9 +7,12 @@
   <xacro:include filename= "$(find ur10e_sim)/urdf/FT_sensor_urdf/net_ft_sensor_macro.urdf.xacro" />
   <xacro:include filename="$(find ur10e_sim)/urdf/pallette.urdf.xacro" />
+  <xacro:include filename="$(find ur10e_sim)/urdf/clamp_for_gripper.urdf.xacro" />
+  <xacro:include filename="$(find ur10e_sim)/urdf/realsense/_d435i.urdf.xacro" />
+  <xacro:include filename="$(find ur10e_sim)/urdf/box.urdf.xacro" />
   <link name="world"/>
   <link name="floor_plate">
     <visual>
       <geometry>
-        <box size="1.0 1.0 0.1"/>
+        <box size="0.8 0.8 0.25"/>
         </geometry>
       <material name="grey">
@@ -19,5 +22,5 @@
     <collision>
       <geometry>
-        <box size="1.0 1.0 0.1"/>
+        <box size="0.8 0.8 0.25"/>
       </geometry>
     </collision>
@@ -31,5 +34,5 @@
     <parent link="world"/>
     <child link="floor_plate"/>
-    <origin xyz="0 0 0.05" rpy="0 0 0"/>
+    <origin xyz="0 0 0.125" rpy="0 0 0"/>
   </joint>
   <xacro:ur_robot
@@ -42,5 +45,5 @@
   <joint name="table_to_robot" type="fixed">
     <parent link="floor_plate"/>
-    <child link="base_link"/> <origin xyz="0 0 0.05" rpy="0 0 0"/>
+    <child link="base_link"/> <origin xyz="0 0 0.125" rpy="0 0 0"/>
   </joint>
   <gazebo reference="table_to_robot">
@@ -64,4 +67,13 @@
     <origin xyz="0 0 0.15" rpy="0 0 0"/>
   </joint>
+  <xacro:clamp_for_gripper prefix=""/>
+  <joint name="clamp_attachment" type="fixed">
+    <parent link="tool0"/>
+    <child link="clamp_base_link"/>
+    <origin xyz="0 -0.018 0.17" rpy="1.57 -1.57 0"/>
+  </joint>
+  <xacro:sensor_d435i parent="camera_mount_link" name="camera" use_nominal_extrinsics="true">
+      <origin xyz="0 0 0" rpy="0 0 0"/>
+    </xacro:sensor_d435i>
   <xacro:wooden_table prefix="right_"/>
   <joint name="right_table_attachment" type="fixed">
@@ -78,8 +90,17 @@
   <xacro:wooden_pallette prefix=""/>
   <joint name="pallette_attachment" type="fixed">
-    <parent link="right_pallette_mount_link"/>
+    <parent link="right_table_mount_link"/>
     <child link="pallette"/>
     <origin xyz="0 0 0" rpy="0 0 0"/>
   </joint>
+  <xacro:table_accessories prefix=""/>
+  <joint name="pedestal_attachment" type="fixed">
+    <parent link="left_table_mount_link"/>
+    <child link="pedestal_link"/>
+    <origin xyz="0 0 0.0" rpy="0 0 0"/>
+  </joint>
+  <gazebo>
+  <disable_collision link1="onrobot_rg2_base_link" link2="clamp_base_link" />
+  </gazebo>
 <gazebo>
   <plugin name="gazebo_ros_link_attacher" filename="libgazebo_ros_link_attacher.so"/>
@@ -90,4 +111,5 @@
     <robotNamespace>/</robotNamespace>
     <robotSimType>gazebo_ros_control/DefaultRobotHWSim</robotSimType>
+    <legacyModeNS>false</legacyModeNS>
   </plugin>
 </gazebo>
